Commit message: gz loads, no robot model, no model in rviz

File: src/install/pioneer/share/pioneer/src/robots/pioneer.urdf (robot description, URDF)
Before this commit: robot pioneer3at_body, 19 links, 18 joints
Links:
- link chassis: geometry collision mesh filename=/home/jeremy/Resources/src/pioneer/src/meshes/chassis.dae; visual mesh filename=/home/jeremy/Resources/src/pioneer/src/meshes/chassis.dae
- link laser_frame: geometry collision box size=0.01 0.01 0.01; visual mesh filename=/home/jeremy/Resources/src/pioneer/src/meshes/hokuyo1.dae
- link p3at_back_left_axle: geometry collision box size=0.01 0.01 0.01; visual mesh filename=/home/jeremy/Resources/src/pioneer/src/meshes/p3at_meshes/a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
- link p3at_back_left_hub: geometry collision box size=0.01 0.01 0.01; visual mesh filename=/home/jeremy/Resources/src/pioneer/src/meshes/p3at_meshes/l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
- link p3at_back_left_wheel: geometry collision mesh filename=/home/jeremy/Resources/src/pioneer/src/meshes/p3at_meshes/w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; visual mesh filename=/home/jeremy/Resources/src/pioneer/src/meshes/p3at_meshes/w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
- link p3at_back_right_axle: geometry collision box size=0.01 0.01 0.01; visual mesh filename=/home/jeremy/Resources/src/pioneer/src/meshes/p3at_meshes/a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
- link p3at_back_right_hub: geometry collision box size=0.01 0.01 0.01; visual mesh filename=/home/jeremy/Resources/src/pioneer/src/meshes/p3at_meshes/r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
- link p3at_back_right_wheel: geometry collision mesh filename=/home/jeremy/Resources/src/pioneer/src/meshes/p3at_meshes/w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; visual mesh filename=/home/jeremy/Resources/src/pioneer/src/meshes/p3at_meshes/w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
- link p3at_front_left_axle: geometry collision box size=0.01 0.01 0.01; visual mesh filename=/home/jeremy/Resources/src/pioneer/src/meshes/p3at_meshes/a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
- link p3at_front_left_hub: geometry collision box size=0.01 0.01 0.01; visual mesh filename=/home/jeremy/Resources/src/pioneer/src/meshes/p3at_meshes/l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
- link p3at_front_left_wheel: geometry collision mesh filename=/home/jeremy/Resources/src/pioneer/src/meshes/p3at_meshes/w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; visual mesh filename=/home/jeremy/Resources/src/pioneer/src/meshes/p3at_meshes/w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
- link p3at_front_right_axle: geometry collision box size=0.01 0.01 0.01; visual mesh filename=/home/jeremy/Resources/src/pioneer/src/meshes/p3at_meshes/a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
- link p3at_front_right_hub: geometry collision box size=0.01 0.01 0.01; visual mesh filename=/home/jeremy/Resources/src/pioneer/src/meshes/p3at_meshes/l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
- link p3at_front_right_wheel: geometry collision mesh filename=/home/jeremy/Resources/src/pioneer/src/meshes/p3at_meshes/w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; visual mesh filename=/home/jeremy/Resources/src/pioneer/src/meshes/p3at_meshes/w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
- link top_plate: geometry collision box size=0.1 0.1 0.1; visual mesh filename=/home/jeremy/Resources/src/pioneer/src/meshes/top.dae

Commit message: gazebo and rviz loading robot

File: src/install/pioneer/share/pioneer/src/robots/pioneer.urdf (robot description, URDF)
Before this commit: robot pioneer3at_body, 19 links, 18 joints
Links:
- link chassis: geometry collision mesh filename=file://$(find pioneer)/src/meshes/chassis.dae; visual mesh filename=file://$(find pioneer)/src/meshes/chassis.dae
- link laser_frame: mass 1e-5 -> 0.1; geometry collision box size=0.1 0.1 0.1; visual mesh filename=file://$(find pioneer)/src/description/meshes/hokuyo1.dae
- link p3at_back_left_axle: geometry collision box size=0.01 0.01 0.01; visual mesh filename=file://$(find pioneer)/src/meshes/p3at_meshes/axle.dae
- link p3at_back_left_hub: geometry collision box size=0.01 0.01 0.01; visual mesh filename=file://$(find pioneer)/src/meshes/p3at_meshes/left_hubcap.d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
- link p3at_back_left_wheel: geometry collision mesh filename=file://$(find pioneer)/src/meshes/p3at_meshes/wheel.dae; visual mesh filename=file://$(find pioneer)/src/meshes/p3at_meshes/wheel.dae
- link p3at_back_right_axle: geometry collision box size=0.01 0.01 0.01; visual mesh filename=file://$(find pioneer)/src/meshes/p3at_meshes/axle.dae
- link p3at_back_right_hub: geometry collision box size=0.01 0.01 0.01; visual mesh filename=file://$(find pioneer)/src/meshes/p3at_meshes/right_hubcap.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
- link p3at_back_right_wheel: geometry collision mesh filename=file://$(find pioneer)/src/meshes/p3at_meshes/wheel.dae; visual mesh filename=file://$(find pioneer)/src/meshes/p3at_meshes/wheel.dae
- link p3at_front_left_axle: geometry collision box size=0.01 0.01 0.01; visual mesh filename=file://$(find pioneer)/src/meshes/p3at_meshes/axle.dae
- link p3at_front_left_hub: geometry collision box size=0.01 0.01 0.01; visual mesh filename=file://$(find pioneer)/src/meshes/p3at_meshes/left_hubcap.d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
- link p3at_front_left_wheel: geometry collision mesh filename=file://$(find pioneer)/src/meshes/p3at_meshes/wheel.dae; visual mesh filename=file://$(find pioneer)/src/meshes/p3at_meshes/wheel.dae
- link p3at_front_right_axle: geometry collision box size=0.01 0.01 0.01; visual mesh filename=file://$(find pioneer)/src/meshes/p3at_meshes/axle.dae
- link p3at_front_right_hub: geometry collision box size=0.01 0.01 0.01; visual mesh filename=file://$(find pioneer)/src/meshes/p3at_meshes/left_hubcap.d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
- link p3at_front_right_wheel: geometry collision mesh filename=file://$(find pioneer)/src/meshes/p3at_meshes/wheel.dae; visual mesh filename=file://$(find pioneer)/src/meshes/p3at_meshes/wheel.dae
- link top_plate: geometry collision box size=0.1 0.1 0.1; visual mesh filename=file://$(find pioneer)/src/meshes/top.dae
Joints:
- joint laser_joint: origin xyz=0.2 0 0.104 rpy=0 0 0 -> xyz=0.043 0 0.254 rpy=0 0 0; parent chassis -> base_link
